Commit message: Add perception code and build&devel for catkin backup

File: src/cr5_description/urdf/camera.xacro (robot description, xacro)
@@ -1,8 +1,9 @@
 <robot name="camera" xmlns:xacro="http://wiki.ros.org/xacro">
+    <xacro:include filename="$(find cr5_description)/urdf/inertia.xacro" />
     <xacro:property name="camera_length" value="0.01" />
     <xacro:property name="camera_width" value="0.025" />
     <xacro:property name="camera_height" value="0.025" />
-    <xacro:property name="camera_x" value="0.08" />
-    <xacro:property name="camera_y" value="0.0" />
+    <xacro:property name="camera_x" value="-1.0" />
+    <xacro:property name="camera_y" value="0" />
     <xacro:property name="camera_z" value="1.0" />
     <xacro:property name="camera_m" value="0.01" />
@@ -10,5 +11,5 @@
         <visual>
             <geometry>
-                <box size="${camera_length} ${camera_width} ${camera_height}" />
+                <mesh filename="package://cr5_description/meshes/kinect/meshes/kinect.dae" />
             </geometry>
             <origin xyz="0.0 0.0 0.0" rpy="0.0 0.0 0.0" />
@@ -29,5 +30,5 @@
     </joint>
     <gazebo reference="camera">
-        <material>Gazebo/Blue</material>
+        <material>Gazebo/Black</material>
     </gazebo>
 </robot>

File: src/cr5_description/urdf/kinect_sensors.xacro (robot description, xacro)
@@ -1,23 +1,109 @@
-<robot name="kinect_sensors" xmlns:xacro="http://wiki.ros.org/xacro">
-  <xacro:include filename="$(find cr5_description)/urdf/inertia.xacro" />
-  <xacro:property name="camera_length" value="0.073000" />
-  <xacro:property name="camera_width" value="0.276000" />
-  <xacro:property name="camera_height" value="0.072000" />
-  <xacro:property name="camera_m" value="0.1" />
-  <link name="kinect_link">
-    <!-- <inertial>
-      <xacro:Box_inertial_matrix m="${camera_m}" l="${camera_length}" w="${camera_width}" h="${camera_height}" />
-    </inertial> -->
-    <collision name="collision">
+<?xml version="1.0"?>
+<robot name="sensor_kinect" xmlns:xacro="http://ros.org/wiki/xacro">
+  <xacro:property name="cam_px" value="-1.3" />
+  <xacro:property name="cam_pz" value="0.7" />
+  <xacro:property name="cam_py" value="-1" />
+	<xacro:property name="cam_or" value="0" />
+	<xacro:property name="cam_op" value="0" />
+	<xacro:property name="cam_oy" value="0.78" />
+  <xacro:property name="kinect_cam_py" value="-0.0125"/>
+  <xacro:property name="M_PI" value="3.14" />
+  <!-- Parameterised in part by the values in turtlebot_properties.urdf.xacro -->
+  <!-- <xacro:macro name="sensor_kinect" params="parent"> -->
+  <link name="camera_rgb_frame"/>
+  <joint name="camera_rgb_joint" type="fixed">
+    <origin xyz="${cam_px} ${cam_py} ${cam_pz}" rpy="${cam_or} ${cam_op} ${cam_oy}"/>
+    <parent link="base_link"/>
+    <child link="camera_rgb_frame" />
+  </joint>
+  <joint name="camera_rgb_optical_joint" type="fixed">
+    <origin xyz="0 0 0" rpy="${-M_PI/2} 0 ${-M_PI/2}" />
+    <parent link="camera_rgb_frame" />
+    <child link="camera_rgb_optical_frame" />
+  </joint>
+  <link name="camera_rgb_optical_frame"/>
+  <joint name="camera_joint" type="fixed">
+    <origin xyz="-0.031 ${-kinect_cam_py} -0.016" rpy="0 0 0"/>
+    <parent link="camera_rgb_frame"/>
+    <child link="camera_link"/>
+  </joint>
+    <link name="camera_link">
+    <visual>
+      <origin xyz="0 0 0" rpy="0 0 0"/>
       <geometry>
-        <box size = "${camera_length} ${camera_width} ${camera_height}"/>
-        <origin xyz="0.0 0.0 0.0" rpy="0.0 0.0 0.0" />
+        <mesh filename="package://cr5_description/meshes/kinect/meshes/kinect.dae"/>
+      </geometry>
+    </visual>
+    <collision>
+      <origin xyz="0.0 0.0 0.0" rpy="0 0 0"/>
+      <geometry>
+        <box size="0.07271 0.27794 0.073"/>
       </geometry>
     </collision>
-    <visual name="visual">
-      <geometry>
-        <mesh filename="$(find cr5_description)/meshes/kinect/meshes/kinect.dae" />
-      </geometry>
-    </visual>
+    <inertial>
+      <mass value="0.564" />
+      <origin xyz="0 0 0" />
+      <inertia ixx="0.003881243" ixy="0.0" ixz="0.0"
+                iyy="0.000498940" iyz="0.0"
+                izz="0.003879257" />
+    </inertial>
   </link>
+    <!-- The fixed joints & links below are usually published by static_transformers launched by the OpenNi launch
+         files. However, for Gazebo simulation we need them, so we add them here.
+         (Hence, don't publish them additionally!) -->
+	<joint name="camera_depth_joint" type="fixed">
+	  <origin xyz="0 ${2 * -kinect_cam_py} 0" rpy="0 0 0" />
+	  <parent link="camera_rgb_frame" />
+	  <child link="camera_depth_frame" />
+	</joint>
+	<link name="camera_depth_frame"/>
+	<joint name="camera_depth_optical_joint" type="fixed">
+	  <origin xyz="0 0 0" rpy="${-M_PI/2} 0 ${-M_PI/2}" />
+	  <parent link="camera_depth_frame" />
+	  <child link="camera_depth_optical_frame" />
+	</joint>
+	<link name="camera_depth_optical_frame"/>
+  <gazebo reference="camera_link">
+    <sensor type="depth" name="camera">
+      <always_on>true</always_on>
+      <update_rate>30.0</update_rate>
+      <camera>
+      <horizontal_fov>${90.0*M_PI/180.0}</horizontal_fov>
+        <image>
+          <format>B8G8R8</format>
+          <width>640</width>
+          <height>480</height>
+        </image>
+        <clip>
+          <near>0.05</near>
+          <far>30.0</far>
+        </clip>
+      </camera>
+      <plugin name="kinect_camera_controller" filename="libgazebo_ros_openni_kinect.so">
+        <cameraName>camera</cameraName>
+        <alwaysOn>true</alwaysOn>
+<!-- Keep this zero, update_rate in the parent <sensor> tag will control the frame rate. -->
+        <updateRate>0</updateRate>
+        <imageTopicName>color/image_raw</imageTopicName>
+        <depthImageTopicName>depth/depth_registered</depthImageTopicName>
+        <pointCloudTopicName>depth_registered/points</pointCloudTopicName>
+        <cameraInfoTopicName>/rgb_raw/camera_info</cameraInfoTopicName>
+        <depthImageCameraInfoTopicName>/depth/camera_info</depthImageCameraInfoTopicName>
+        <frameName>camera_depth_optical_frame</frameName>
+        <pointCloudCutoff>0.125</pointCloudCutoff>
+        <pointCloudCutoffMax>5.0</pointCloudCutoffMax>
+        <baseline>0.1</baseline>
+        <distortion_k1>0.0</distortion_k1>
+        <distortion_k2>0.0</distortion_k2>
+        <distortion_k3>0.0</distortion_k3>
+        <distortion_t1>0.0</distortion_t1>
+        <distortion_t2>0.0</distortion_t2>
+        <CxPrime>0</CxPrime>
+        <Cx>0</Cx>
+        <Cy>0</Cy>
+        <focalLength>0</focalLength>
+        <hackBaseline>0</hackBaseline>
+      </plugin>
+    </sensor>
+  </gazebo>
 </robot>

File: src/cr5_description/urdf/robot_with_kinect.xacro (robot description, xacro)
@@ -5,54 +5,3 @@
     <!-- <xacro:include filename="$(find cr5_description)/urdf/cr5.urdf.xacro" />   -->
     <xacro:include filename="$(find cr5_description)/urdf/kinect_sensors.xacro" />
-    <joint name="kinect2base" type="fixed">
-        <parent link="base_link"/>
-        <child link="kinect_link"/>
-        <origin xyz="1.5 0 1.0" rpy="0 0 3.14"/>
-    </joint>
-    <!-- 虚拟相机坐标系 -->
-    <link name="rgb"/>
-    <joint name="rgb_joint" type="fixed">
-        <origin xyz="0 0 0.1" rpy="0 0 0"/>
-        <parent link="kinect_link"/>
-        <child link="rgb"/>
-    </joint>
-    <gazebo reference="kinect_link">
-      <material>Gazebo/Black</material>
-  </gazebo>
-  <gazebo reference="kinect_link">
-    <sensor name="camera" type="depth">
-      <always_on>true</always_on>
-      <update_rate>20</update_rate>
-      <camera>
-        <horizontal_fov>1.047198</horizontal_fov>
-        <image>
-          <width>640</width>
-          <height>480</height>
-          <format>R8G8B8</format>
-        </image>
-        <clip>
-          <near>0.05</near>
-          <far>3</far>
-        </clip>
-      </camera>
-      <plugin name="kinect_camera_controller" filename="libgazebo_ros_openni_kinect.so">
-          <cameraName>camera</cameraName>
-          <alwaysOn>true</alwaysOn>
-          <updateRate>30</updateRate>
-          <imageTopicName>rgb/image_raw</imageTopicName>
-          <depthImageTopicName>depth/image_raw</depthImageTopicName>
-          <pointCloudTopicName>depth/points</pointCloudTopicName>
-          <cameraInfoTopicName>rgb/camera_info</cameraInfoTopicName>
-          <depthImageCameraInfoTopicName>depth/camera_info</depthImageCameraInfoTopicName>
-          <frameName>rgb</frameName>
-          <baseline>0.1</baseline>
-          <distortion_k1>0.0</distortion_k1>
-          <distortion_k2>0.0</distortion_k2>
-          <distortion_k3>0.0</distortion_k3>
-          <distortion_t1>0.0</distortion_t1>
-          <distortion_t2>0.0</distortion_t2>
-          <pointCloudCutoff>0.4</pointCloudCutoff>
-        </plugin>
-      </sensor>
-  </gazebo>
 </robot>
