Commit message: Update gazebo simulation

File: src/cr5_description/urdf/cr5_dh.urdf.xacro (robot description, xacro)
@@ -1,4 +1,5 @@
 <?xml version="1.0"?>
 <robot name="cr5" xmlns:xacro="http://ros.org/wiki/xacro">
+  <xacro:include filename="$(find cr5_description)/urdf/inertia.xacro" />
   <link name="base_link">
     <inertial>
@@ -410,4 +411,18 @@
       offset="0" />
   </joint>
+  <xacro:include filename="$(find cr5_description)/urdf/kinect_sensors.xacro" />
+  <joint name="kinect2base" type="fixed">
+    <parent link="base_link"/>
+    <child link="kinect_link"/>
+    <origin xyz="1.5 0 1.0" rpy="0 0 3.14"/>
+  </joint>
+  <!-- 虚拟相机坐标系 -->
+  <link name="rgb"/>
+  <joint name="rgb_joint" type="fixed">
+    <origin xyz="0 0 0.1" rpy="0 0 0"/>
+    <parent link="kinect_link"/>
+    <child link="rgb"/>
+  </joint>
+  <!-- 电机驱动 -->
   <xacro:macro name="transmission_block" params="joint_name">
     <transmission name="tran1">
@@ -432,6 +447,45 @@
   <gazebo>
     <plugin name="gazebo_ros_control" filename="libgazebo_ros_control.so">
-      <robotNamespace>/cr5</robotNamespace>
+      <robotNamespace>/</robotNamespace>
     </plugin>
   </gazebo>
+  <gazebo reference="kinect_link">
+      <material>Gazebo/Black</material>
+  </gazebo>
+  <gazebo reference="kinect_link">
+    <sensor name="camera" type="depth">
+      <always_on>true</always_on>
+      <update_rate>20</update_rate>
+      <camera>
+        <horizontal_fov>1.047198</horizontal_fov>
+        <image>
+          <width>640</width>
+          <height>480</height>
+          <format>R8G8B8</format>
+        </image>
+        <clip>
+          <near>0.05</near>
+          <far>3</far>
+        </clip>
+      </camera>
+      <plugin name="kinect_camera_controller" filename="libgazebo_ros_openni_kinect.so">
+          <cameraName>camera</cameraName>
+          <alwaysOn>true</alwaysOn>
+          <updateRate>30</updateRate>
+          <imageTopicName>rgb/image_raw</imageTopicName>
+          <depthImageTopicName>depth/image_raw</depthImageTopicName>
+          <pointCloudTopicName>depth/points</pointCloudTopicName>
+          <cameraInfoTopicName>rgb/camera_info</cameraInfoTopicName>
+          <depthImageCameraInfoTopicName>depth/camera_info</depthImageCameraInfoTopicName>
+          <frameName>rgb</frameName>
+          <baseline>0.1</baseline>
+          <distortion_k1>0.0</distortion_k1>
+          <distortion_k2>0.0</distortion_k2>
+          <distortion_k3>0.0</distortion_k3>
+          <distortion_t1>0.0</distortion_t1>
+          <distortion_t2>0.0</distortion_t2>
+          <pointCloudCutoff>0.4</pointCloudCutoff>
+        </plugin>
+      </sensor>
+  </gazebo>
 </robot>

Commit message: Update global planner for gp_planner

File: src/cr5_description/urdf/cr5_dh.urdf.xacro (robot description, xacro)
@@ -410,17 +410,4 @@
       multiplier="1"
       offset="0" />
-  </joint>
-  <xacro:include filename="$(find cr5_description)/urdf/kinect_sensors.xacro" />
-  <joint name="kinect2base" type="fixed">
-    <parent link="base_link"/>
-    <child link="kinect_link"/>
-    <origin xyz="1.5 0 1.0" rpy="0 0 3.14"/>
-  </joint>
-  <!-- 虚拟相机坐标系 -->
-  <link name="rgb"/>
-  <joint name="rgb_joint" type="fixed">
-    <origin xyz="0 0 0.1" rpy="0 0 0"/>
-    <parent link="kinect_link"/>
-    <child link="rgb"/>
   </joint>
   <!-- 电机驱动 -->
@@ -450,42 +437,3 @@
     </plugin>
   </gazebo>
-  <gazebo reference="kinect_link">
-      <material>Gazebo/Black</material>
-  </gazebo>
-  <gazebo reference="kinect_link">
-    <sensor name="camera" type="depth">
-      <always_on>true</always_on>
-      <update_rate>20</update_rate>
-      <camera>
-        <horizontal_fov>1.047198</horizontal_fov>
-        <image>
-          <width>640</width>
-          <height>480</height>
-          <format>R8G8B8</format>
-        </image>
-        <clip>
-          <near>0.05</near>
-          <far>3</far>
-        </clip>
-      </camera>
-      <plugin name="kinect_camera_controller" filename="libgazebo_ros_openni_kinect.so">
-          <cameraName>camera</cameraName>
-          <alwaysOn>true</alwaysOn>
-          <updateRate>30</updateRate>
-          <imageTopicName>rgb/image_raw</imageTopicName>
-          <depthImageTopicName>depth/image_raw</depthImageTopicName>
-          <pointCloudTopicName>depth/points</pointCloudTopicName>
-          <cameraInfoTopicName>rgb/camera_info</cameraInfoTopicName>
-          <depthImageCameraInfoTopicName>depth/camera_info</depthImageCameraInfoTopicName>
-          <frameName>rgb</frameName>
-          <baseline>0.1</baseline>
-          <distortion_k1>0.0</distortion_k1>
-          <distortion_k2>0.0</distortion_k2>
-          <distortion_k3>0.0</distortion_k3>
-          <distortion_t1>0.0</distortion_t1>
-          <distortion_t2>0.0</distortion_t2>
-          <pointCloudCutoff>0.4</pointCloudCutoff>
-        </plugin>
-      </sensor>
-  </gazebo>
 </robot>

Commit message: fix handeye and add test code

File: src/cr5_description/urdf/cr5_dh.urdf.xacro (robot description, xacro)
@@ -57,4 +57,12 @@
       </geometry>
     </collision>
+    <!-- 添加Contact Sensor -->
+    <sensor name="Link1_contact_sensor" type="contact">
+      <update_rate>30</update_rate>
+      <contact>
+        <collision>Link1::collision</collision>
+      </contact>
+      <plugin name="contact_plugin" filename="libContactPlugin.so"/>
+    </sensor>
   </link>
   <joint name="joint1" type="revolute">
@@ -92,4 +100,12 @@
       </geometry>
     </collision>
+    <!-- 添加Contact Sensor -->
+    <sensor name="Link2contact_sensor" type="contact">
+      <update_rate>30</update_rate>
+      <contact>
+        <collision>Link2::collision</collision>
+      </contact>
+      <plugin name="contact_plugin" filename="libContactPlugin.so"/>
+    </sensor>
   </link>
   <joint name="joint2" type="revolute">
@@ -127,4 +143,12 @@
       </geometry>
     </collision>
+    <!-- 添加Contact Sensor -->
+    <sensor name="Link3_contact_sensor" type="contact">
+      <update_rate>30</update_rate>
+      <contact>
+        <collision>Link3::collision</collision>
+      </contact>
+      <plugin name="contact_plugin" filename="libContactPlugin.so"/>
+    </sensor>
   </link>
   <joint name="joint3" type="revolute">
@@ -162,4 +186,13 @@
       </geometry>
     </collision>
+    <!-- 添加Contact Sensor -->
+    <sensor name="Link4_contact_sensor" type="contact">
+      <update_rate>30</update_rate>
+      <contact>
+        <collision>Link4::collision</collision>
+      </contact>
+      <plugin name="contact_plugin" filename="libContactPlugin.so"/>
+    </sensor>
+  </link>
   </link>
   <joint name="joint4" type="revolute">
@@ -197,4 +230,13 @@
       </geometry>
     </collision>
+    <!-- 添加Contact Sensor -->
+    <sensor name="Link5_contact_sensor" type="contact">
+      <update_rate>30</update_rate>
+      <contact>
+        <collision>Link5::collision</collision>
+      </contact>
+      <plugin name="contact_plugin" filename="libContactPlugin.so"/>
+    </sensor>
+  </link>
   </link>
   <joint name="joint5" type="revolute">
@@ -232,4 +274,13 @@
       </geometry>
     </collision>
+    <!-- 添加Contact Sensor -->
+    <sensor name="Link6_contact_sensor" type="contact">
+      <update_rate>30</update_rate>
+      <contact>
+        <collision>Link6::collision</collision>
+      </contact>
+      <plugin name="contact_plugin" filename="libContactPlugin.so"/>
+    </sensor>
+  </link>
   </link>
   <joint name="joint6" type="revolute">

File: src/cr5_description/urdf/kinect_sensors.xacro (robot description, xacro)
@@ -3,8 +3,8 @@
   <xacro:property name="cam_px" value="-1.3" />
   <xacro:property name="cam_pz" value="0.7" />
-  <xacro:property name="cam_py" value="-1" />
+  <xacro:property name="cam_py" value="0.8" />
 	<xacro:property name="cam_or" value="0" />
 	<xacro:property name="cam_op" value="0" />
-	<xacro:property name="cam_oy" value="0.78" />
+	<xacro:property name="cam_oy" value="-0.78" />
   <xacro:property name="kinect_cam_py" value="-0.0125"/>
   <xacro:property name="M_PI" value="3.14" />

Commit message: fix cr5_dh_urdf.xacro

File: src/cr5_description/urdf/cr5_dh.urdf.xacro (robot description, xacro)
@@ -195,5 +195,4 @@
     </sensor>
   </link>
-  </link>
   <joint name="joint4" type="revolute">
     <origin xyz="-0.357 0 0.141" rpy="0 0 -1.5708" />
@@ -239,5 +238,4 @@
     </sensor>
   </link>
-  </link>
   <joint name="joint5" type="revolute">
     <origin xyz="0 -0.116 0" rpy="1.5708 0 0" />
@@ -282,5 +280,4 @@
       <plugin name="contact_plugin" filename="libContactPlugin.so"/>
     </sensor>
-  </link>
   </link>
   <joint name="joint6" type="revolute">
