Commit message: fix some problem

File: src/cr5_description/urdf/cr5.urdf.xacro (robot description, xacro)
@@ -2,4 +2,5 @@
 <robot name="cr5" xmlns:xacro="http://ros.org/wiki/xacro">
   <!-- Robot Model URDF -->
+  <xacro:include filename="$(find cr5_description)/urdf/inertia.xacro" />
   <link name="base_link">
     <inertial>
@@ -57,4 +58,12 @@
       </geometry>
     </collision>
+    <!-- 添加Contact Sensor -->
+    <sensor name="Link1_contact_sensor" type="contact">
+      <update_rate>30</update_rate>
+      <contact>
+        <collision>Link1::collision</collision>
+      </contact>
+      <plugin name="contact_plugin" filename="libContactPlugin.so"/>
+    </sensor>
   </link>
   <joint name="joint1" type="revolute">
@@ -92,4 +101,12 @@
       </geometry>
     </collision>
+    <!-- 添加Contact Sensor -->
+    <sensor name="Link2contact_sensor" type="contact">
+      <update_rate>30</update_rate>
+      <contact>
+        <collision>Link2::collision</collision>
+      </contact>
+      <plugin name="contact_plugin" filename="libContactPlugin.so"/>
+    </sensor>
   </link>
   <joint name="joint2" type="revolute">
@@ -127,4 +144,12 @@
       </geometry>
     </collision>
+    <!-- 添加Contact Sensor -->
+    <sensor name="Link3_contact_sensor" type="contact">
+      <update_rate>30</update_rate>
+      <contact>
+        <collision>Link3::collision</collision>
+      </contact>
+      <plugin name="contact_plugin" filename="libContactPlugin.so"/>
+    </sensor>
   </link>
   <joint name="joint3" type="revolute">
@@ -162,4 +187,12 @@
       </geometry>
     </collision>
+    <!-- 添加Contact Sensor -->
+    <sensor name="Link4_contact_sensor" type="contact">
+      <update_rate>30</update_rate>
+      <contact>
+        <collision>Link4::collision</collision>
+      </contact>
+      <plugin name="contact_plugin" filename="libContactPlugin.so"/>
+    </sensor>
   </link>
   <joint name="joint4" type="revolute">
@@ -197,4 +230,12 @@
       </geometry>
     </collision>
+    <!-- 添加Contact Sensor -->
+    <sensor name="Link5_contact_sensor" type="contact">
+      <update_rate>30</update_rate>
+      <contact>
+        <collision>Link5::collision</collision>
+      </contact>
+      <plugin name="contact_plugin" filename="libContactPlugin.so"/>
+    </sensor>
   </link>
   <joint name="joint5" type="revolute">
@@ -232,4 +273,12 @@
       </geometry>
     </collision>
+    <!-- 添加Contact Sensor -->
+    <sensor name="Link6_contact_sensor" type="contact">
+      <update_rate>30</update_rate>
+      <contact>
+        <collision>Link6::collision</collision>
+      </contact>
+      <plugin name="contact_plugin" filename="libContactPlugin.so"/>
+    </sensor>
   </link>
   <joint name="joint6" type="revolute">

File: src/cr5_description/urdf/cr5_dh.urdf.xacro (robot description, xacro)
@@ -485,3 +485,11 @@
     </plugin>
   </gazebo>
+  <gazebo>
+    <plugin name="contact_sensor_plugin" filename="libgazebo_ros_contact.so">
+      <robotNamespace>/gazebo</robotNamespace>
+      <alwaysOn>true</alwaysOn>
+      <updateRate>50.0</updateRate>
+      <contactTopicName>contact</contactTopicName>
+    </plugin>
+  </gazebo>
 </robot>
