Commit message: Add adujstment for init values and opt settings

File: src/cr5_description/urdf/kinect_sensors.xacro (robot description, xacro)
@@ -6,5 +6,5 @@
 	<xacro:property name="cam_or" value="0" />
 	<xacro:property name="cam_op" value="0" />
-	<xacro:property name="cam_oy" value="-0.78" />
+	<xacro:property name="cam_oy" value="-0.9" />
   <xacro:property name="kinect_cam_py" value="-0.0125"/>
   <xacro:property name="M_PI" value="3.14" />
